File: keylime_pcb/bank14.kicad_sch (KiCad schematic)
At the start: 0 parts

Commit message: Finished adding most components.
Parts:
- added D1, D2: LED_ABGR, symbol Device:LED_ABGR
- added R4, R5: 100, symbol Device:R
- added U1: xc7s15cpga196, symbol xilinx7:xc7s15cpga196
Connections:
- new net: D1.1 (A), R4.2
- new net: D1.2 (BK), U1.D11 (IO_L9N_T1_DQS_D13_14)
- new net: D1.3 (GK), U1.E12 (IO_L10N_T1_D15_14)
- new net: D1.4 (RK), U1.F13 (IO_L11N_T1_SRCC_14)
- new net: U1.F10 (VCCO_14[3]), U1.H10 (VCCO_14[3]), U1.K10 (VCCO_14[3])
- new net: D2.2 (BK), U1.J13 (IO_L14P_T2_SRCC_14)
- new net: D2.3 (GK), U1.J14 (IO_L15P_T2_DQS_RDWR_B_14)
- new net: D2.4 (RK), U1.K11 (IO_L16P_T2_CSI_B_14)
- new net: D2.1 (A), R5.2
- new net GND: U1.B10 (IO_L3P_T0_DQS_PUDC_B_14)
- new net QSPI_CS: U1.D13 (IO_L6P_T0_FCS_B_14)
- new net QSPI_DQ0: U1.C10 (IO_L1P_T0_D00_MOSI_14)
- new net QSPI_DQ1: U1.C11 (IO_L1N_T0_D01_DIN_14)
- new net QSPI_DQ2: U1.B11 (IO_L2P_T0_D02_14)
- new net QSPI_DQ3: U1.A12 (IO_L2N_T0_D03_14)
- new net UART_RX: U1.L13 (IO_L18N_T2_D27_14)
- new net UART_TX: U1.L12 (IO_L18P_T2_D28_14)
- new net VCC3V3: R4.1, R5.1
