File: keylime_pcb/bank34.kicad_sch (KiCad schematic)
At the start: 0 parts

Commit message: Finished adding most components.
Parts:
- added U1: xc7s15cpga196, symbol xilinx7:xc7s15cpga196
Connections:
- new net: U1.E5 (VCCO_34[3]), U1.G5 (VCCO_34[3]), U1.J5 (VCCO_34[3])
